File: cbEval.ATtiny412_1614.kicad_sch (KiCad schematic)
At the start: 59 parts, among them J1 Bergstik-II_3, J11 Bergstik-II_3, J12 Bergstik-II_3, J13 Bergstik-II_6, J14 Bergstik-II_6, J15 Bergstik-II_6, J16 Bergstik-II_3, J17 Bergstik-II_6, J18 Bergstik-II_3, J19 Bergstik-II_6, J2 Bergstik-II_6, J20 Bergstik-II_3, J21 Bergstik-II_3, J22 Bergstik-II_2, J23 Bergstik-II_2, J3 Header.Hor.2x8.9-103326-0-08, J4 Header.Hor.2x8.9-103326-0-08, J5 Socket.Hor.2x8.1-5535512-8, J6 Socket.Hor.2x8.1-5535512-8, J7 Bergstik-II_3, J8 Bergstik-II_2, U1 ATtiny412-SSFR, U2 ATtiny1614-SSFR

Commit message: PowerBus-Belegung V1.1
Connections:
- net +15V: now also J4.4, J5.4; no longer J4.5, J5.5
- net +3V3: now also J4.3, J5.3; no longer J4.4, J5.4
- net +5V: now also J4.5, J5.5; no longer J4.3, J5.3
- net SPI-~CE renamed SPI-~{CE}
Other:
- moved on the sheet: H1
Changed lines of the file:
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@@
-(kicad_sch (version 20210126) (generator eeschema)
+(kicad_sch (version 20210621) (generator eeschema)
   (paper "A4")
   (title_block
     (title "cbEval ATtiny412 & ATtiny1614")
-    (rev "1.0.0")
+    (rev "1.1.0")
   )
   (junction (at 35.56 48.26) (diameter 0.9144) (color 0 0 0 0))
@@
   (junction (at 48.26 93.98) (diameter 0.9144) (color 0 0 0 0))
   (junction (at 50.8 124.46) (diameter 0.9144) (color 0 0 0 0))
-  (junction (at 50.8 137.16) (diameter 0.9144) (color 0 0 0 0))
+  (junction (at 50.8 142.24) (diameter 0.9144) (color 0 0 0 0))
   (junction (at 55.88 76.2) (diameter 0.9144) (color 0 0 0 0))
   (junction (at 58.42 78.74) (diameter 0.9144) (color 0 0 0 0))
@@
   (junction (at 60.96 167.64) (diameter 0.9144) (color 0 0 0 0))
   (junction (at 66.04 124.46) (diameter 0.9144) (color 0 0 0 0))
-  (junction (at 66.04 139.7) (diameter 0.9144) (color 0 0 0 0))
+  (junction (at 66.04 137.16) (diameter 0.9144) (color 0 0 0 0))
   (junction (at 73.66 66.04) (diameter 0.9144) (color 0 0 0 0))
   (junction (at 81.28 124.46) (diameter 0.9144) (color 0 0 0 0))
-  (junction (at 81.28 142.24) (diameter 0.9144) (color 0 0 0 0))
+  (junction (at 81.28 139.7) (diameter 0.9144) (color 0 0 0 0))
   (junction (at 86.36 30.48) (diameter 0.9144) (color 0 0 0 0))
   (junction (at 86.36 68.58) (diameter 0.9144) (color 0 0 0 0))
@@
     (stroke (width 0) (type solid) (color 0 0 0 0))
   )
-  (wire (pts (xy 33.02 137.16) (xy 50.8 137.16))
-    (stroke (width 0) (type solid) (color 0 0 0 0))
-  )
-  (wire (pts (xy 33.02 139.7) (xy 66.04 139.7))
-    (stroke (width 0) (type solid) (color 0 0 0 0))
-  )
-  (wire (pts (xy 33.02 142.24) (xy 81.28 142.24))
+  (wire (pts (xy 33.02 137.16) (xy 66.04 137.16))
+    (stroke (width 0) (type solid) (color 0 0 0 0))
+  )
+  (wire (pts (xy 33.02 139.7) (xy 81.28 139.7))
+    (stroke (width 0) (type solid) (color 0 0 0 0))
+  )
+  (wire (pts (xy 33.02 142.24) (xy 50.8 142.24))
     (stroke (width 0) (type solid) (color 0 0 0 0))
   )
@@
     (stroke (width 0) (type solid) (color 0 0 0 0))
   )
-  (wire (pts (xy 50.8 124.46) (xy 50.8 137.16))
-    (stroke (width 0) (type solid) (color 0 0 0 0))
-  )
-  (wire (pts (xy 50.8 137.16) (xy 114.3 137.16))
+  (wire (pts (xy 50.8 124.46) (xy 50.8 142.24))
+    (stroke (width 0) (type solid) (color 0 0 0 0))
+  )
+  (wire (pts (xy 50.8 142.24) (xy 114.3 142.24))
     (stroke (width 0) (type solid) (color 0 0 0 0))
   )
@@
     (stroke (width 0) (type solid) (color 0 0 0 0))
   )
-  (wire (pts (xy 66.04 124.46) (xy 66.04 139.7))
-    (stroke (width 0) (type solid) (color 0 0 0 0))
-  )
-  (wire (pts (xy 66.04 139.7) (xy 114.3 139.7))
+  (wire (pts (xy 66.04 124.46) (xy 66.04 137.16))
+    (stroke (width 0) (type solid) (color 0 0 0 0))
+  )
+  (wire (pts (xy 66.04 137.16) (xy 114.3 137.16))
     (stroke (width 0) (type solid) (color 0 0 0 0))
   )
@@
     (stroke (width 0) (type solid) (color 0 0 0 0))
   )
-  (wire (pts (xy 81.28 124.46) (xy 81.28 142.24))
-    (stroke (width 0) (type solid) (color 0 0 0 0))
-  )
-  (wire (pts (xy 81.28 142.24) (xy 114.3 142.24))
+  (wire (pts (xy 81.28 124.46) (xy 81.28 139.7))
+    (stroke (width 0) (type solid) (color 0 0 0 0))
+  )
+  (wire (pts (xy 81.28 139.7) (xy 114.3 139.7))
     (stroke (width 0) (type solid) (color 0 0 0 0))
   )
@@
     (effects (font (size 1.27 1.27)) (justify left bottom))
   )
-  (label "SPI-~CE" (at 38.1 73.66 0)
+  (label "SPI-~{CE}" (at 38.1 73.66 0)
     (effects (font (size 1.27 1.27)) (justify left bottom))
   )
@@
     (effects (font (size 1.27 1.27)) (justify left bottom))
   )
-  (label "~RESET" (at 66.04 149.86 0)
+  (label "~{RESET}" (at 66.04 149.86 0)
     (effects (font (size 1.27 1.27)) (justify left bottom))
   )
@@
     (effects (font (size 1.27 1.27)) (justify left bottom))
   )
-  (label "~RESET" (at 104.14 180.34 0)
+  (label "~{RESET}" (at 104.14 180.34 0)
     (effects (font (size 1.27 1.27)) (justify left bottom))
   )
@@
     (effects (font (size 1.27 1.27)) (justify left bottom))
   )
-  (label "SPI-~CE" (at 129.54 73.66 0)
+  (label "SPI-~{CE}" (at 129.54 73.66 0)
     (effects (font (size 1.27 1.27)) (justify left bottom))
   )
@@
     (effects (font (size 1.27 1.27)) (justify left bottom))
   )
-  (label "SPI-~CE" (at 129.54 99.06 0)
+  (label "SPI-~{CE}" (at 129.54 99.06 0)
     (effects (font (size 1.27 1.27)) (justify left bottom))
   )
@@
     (pin "2")
   )
-  (symbol (lib_id "H.Housing:CIME.E.BE3500S.1x") (at -5.08 20.32 0) (unit 1)
-    (in_bom yes) (on_board yes)
-    (property "Reference" "H1" (id 0) (at -7.62 27.94 0)
-      (effects (font (size 1.27 1.27)) (justify left))
-    )
-    (property "Value" "CIME.E.BE3500S.1x" (id 1) (at -7.62 30.48 0)
-      (effects (font (size 1.27 1.27)) (justify left))
-    )
-    (property "Footprint" "BTech.Housing:Camdenboss.CIME.E.BE3500S.1x" (id 2) (at -5.08 12.7 0)
-      (effects (font (size 1.016 1.016)) hide)
-    )
-    (property "Datasheet" "https://cdn-reichelt.de/documents/datenblatt/C700/CIME_E.pdf" (id 3) (at -5.08 10.16 0)
-      (effects (font (size 1.016 1.016)) hide)
-    )
-    (property "ID" "CIME/E/BE3500S" (id 4) (at -5.08 20.32 90)
+  (symbol (lib_id "H.Housing:CIME.E.BE3500S.1x") (at 256.54 20.32 0) (unit 1)
+    (in_bom yes) (on_board yes)
+    (property "Reference" "H1" (id 0) (at 261.62 17.78 0)
+      (effects (font (size 1.27 1.27)) (justify left))
+    )
+    (property "Value" "CIME.E.BE3500S.1x" (id 1) (at 261.62 20.32 0)
+      (effects (font (size 1.27 1.27)) (justify left))
+    )
+    (property "Footprint" "BTech.Housing:Camdenboss.CIME.E.BE3500S.1x" (id 2) (at 256.54 12.7 0)
+      (effects (font (size 1.016 1.016)) hide)
+    )
+    (property "Datasheet" "https://cdn-reichelt.de/documents/datenblatt/C700/CIME_E.pdf" (id 3) (at 256.54 10.16 0)
+      (effects (font (size 1.016 1.016)) hide)
+    )
+    (property "ID" "CIME/E/BE3500S" (id 4) (at 256.54 20.32 90)
       (effects (font (size 0.635 0.635) italic))
     )
